File: usb-led.brd (EAGLE design)
At the start: 41.9 x 12 mm, 13 parts, among them U1 Tiny85-20-SMT

Commit message: 0.0.0.1 => add ground planes to ground
Routing:
- net GND: track 87.5 -> 0.00 mm, vias 1 -> 0
- net DIN_2: track 11.1 -> 29.2 mm
- net VCC: track 80.9 -> 66.4 mm, vias 3 -> 1
- net SCK: track 19.3 -> 12.2 mm
- net MOSI/DIN: track 26.5 -> 21.4 mm, vias 0 -> 1
- net USB_D_PLUS_RAW: track 18.6 -> 21.9 mm
- net USB_D_MINUS_RAW: track 18.6 -> 20.5 mm
- net MISO: track 13.8 -> 15.6 mm, vias 0 -> 1
- net USB_D_MINUS: track 12.6 -> 13.2 mm
- added copper zone on layer 1, net GND
- added copper zone on layer 16, net GND
- removed copper zone on layer 1, net N$2
- removed copper zone on layer 16, net N$3
Other:
- board text added: "v0.0.0.1"
- board text removed: "v0.0.1"
