File: hardware/apa102/weblight_developer.brd (EAGLE design)
At the start: 43.2 x 12 mm, 14 parts, among them U1 ATTiny85-20SU

Commit message: a-osh1
Parts:
- removed SW_RESET: BUTTON_TD-85XU, weblight:BUTTON_TD-85XU
- added ICSP1: AVR_SPI_PRG_62X3_LOCK, SparkFun-Connectors:2X3_LOCK
- added ICSP2: POGOPIN-CONNWITHVIAS, weblight:POGOPROG-CONN-0H
- added SW1: TACT_2PIN, weblight:TD-85XU
- JP1: value AVR_SPI_PRG_62X3_LOCK -> LED_OUT; device SparkFun-Connectors:2X3_LOCK -> microbuilder:1X04_ROUND
- R4: value 470 -> 4.7K
- moved R3 9.55 mm to (15.2, 2.54)
- moved D1 6.60 mm to (14.0, 9.65), turned to 90 degrees
- moved R1 6.51 mm to (11.4, 9.65)
- moved R2 6.38 mm to (12.7, 2.54)
- moved C1 6.08 mm to (26.8, 9.14)
- moved JP1 4.45 mm to (38.7, 5.71)
- moved C2 1.42 mm to (29.3, 9.14)
- moved LED2 1.15 mm to (34.2, 3.05)
- moved LED1 1.14 mm to (34.2, 8.89)
- moved D2 0.99 mm to (15.9, 9.65)
- moved U1 0.77 mm to (19.8, 6.86)
- moved R4 0.68 mm to (24.1, 9.14)
Connections:
- net DIN_2 renamed DATA_2
- net SCK_2 renamed CLK_2
- removed net DIN_1: LED1.DI, R4.2
- removed net MOSI/DIN_RAW: JP1.4, R4.1, U1.5
- removed net RESET: JP1.5, SW_RESET.PAD1, U1.1
- removed net SCK_1: JP1.3, LED1.CI, U1.7
- new net CLK_1/SCK: ICSP1.3, ICSP2.4, LED1.CI, U1.7
- new net CLK_3: JP1.2, LED2.CO
- new net DATA_1/MOSI: ICSP1.4, ICSP2.2, LED1.DI, U1.5
- new net DATA_3: JP1.3, LED2.DO
- new net N_RESET: ICSP1.5, ICSP2.1, R4.1, SW1.P$1, U1.1
- net GND: now also ICSP1.6, ICSP2.5, JP1.4, SW1.P$2; no longer JP1.6, SW_RESET.PAD2
- net MISO: now also ICSP1.1, ICSP2.3; no longer JP1.1
- net VCC: now also ICSP1.2, ICSP2.6, JP1.1, R4.2; no longer JP1.2
Routing:
- net DATA_1/MOSI: track 0.00 -> 46.7 mm, vias 0 -> 2
- net N_RESET: track 0.00 -> 43.2 mm, vias 0 -> 1
- net CLK_1/SCK: track 0.00 -> 32.1 mm, vias 0 -> 1
- net SCK_1: track 31.4 -> 0.00 mm
- net MOSI/DIN_RAW: track 25.6 -> 0.00 mm
- net RESET: track 25.4 -> 0.00 mm
- net USB_D_MINUS_RAW: track 40.8 -> 21.6 mm
- net VCC: track 74.3 -> 85.4 mm, vias 5 -> 4
- net MISO: track 23.3 -> 34.3 mm, vias 1 -> 2
- net GND: track 85.5 -> 77.3 mm, vias 1 -> 2
- net CLK_3: track 0.00 -> 7.57 mm
- net DIN_1: track 6.75 -> 0.00 mm
- net DATA_3: track 0.00 -> 2.74 mm
- net USB_D_MINUS: track 7.49 -> 5.13 mm
- net USB_D_PLUS: track 11.0 -> 9.65 mm
- added copper zone on layer 1, net GND
- added copper zone on layer 16, net GND
- removed copper zone on layer 16, net N$1
- removed copper zone on layer 1, net N$2
Other:
- board size 43.2 x 12 mm -> 48.3 x 12 mm
- board text added: "GND DO CO VCC"
