File: hardware/weblight_developer.brd (EAGLE design)
At the start: 48.3 x 12 mm, 16 parts, among them SW1 TACT_2PIN, U1 ATTiny85-20SU

Commit message: NRES pullup 10K; big cap 1uF
Parts:
- C1: value 10uF -> 1uF
- R4: value 4.7K -> 10K
Changed lines of the file:
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@@
 <?xml version="1.0" encoding="utf-8"?>
 <!DOCTYPE eagle SYSTEM "eagle.dtd">
-<eagle version="7.4.0">
+<eagle version="7.5.0">
 <drawing>
 <settings>
@@
 </autorouter>
 <elements>
-<element name="C1" library="rcl" package="C0805" value="10uF" x="26.797" y="9.144" smashed="yes" rot="R270">
+<element name="C1" library="rcl" package="C0805" value="1uF" x="26.797" y="9.144" smashed="yes" rot="R270">
 <attribute name="NAME" x="26.67" y="7.112" size="0.8128" layer="25" font="vector" rot="R90" align="center-right"/>
 <attribute name="VALUE" x="24.257" y="10.414" size="1.27" layer="27" rot="R270"/>
@@
 <attribute name="NAME" x="18.669" y="4.953" size="0.8128" layer="25" font="vector" rot="R90"/>
 </element>
-<element name="R4" library="rcl" package="R0805" value="4.7K" x="24.13" y="9.144" smashed="yes" rot="R90">
+<element name="R4" library="rcl" package="R0805" value="10K" x="24.13" y="9.144" smashed="yes" rot="R90">
 <attribute name="NAME" x="24.13" y="7.112" size="0.8128" layer="25" font="vector" rot="R90" align="center-right"/>
 <attribute name="VALUE" x="26.035" y="8.509" size="1.27" layer="27" rot="R90"/>
