File: hardware/weblight_developer.sch (EAGLE design)
At the start: 16 parts, among them SW1 TACT_2PIN, U1 ATTiny85-20SU

Commit message: NRES pullup 10K; big cap 1uF
Parts:
- C1: value 10uF -> 1uF
- R4: value 4.7K -> 10K
Changed lines of the file:
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@@
 <?xml version="1.0" encoding="utf-8"?>
 <!DOCTYPE eagle SYSTEM "eagle.dtd">
-<eagle version="7.4.0">
+<eagle version="7.5.0">
 <drawing>
 <settings>
@@
 <parts>
 <part name="JP-USB-TOP" library="SparkFun-Connectors" deviceset="USB" device="PCB"/>
-<part name="C1" library="rcl" deviceset="C-US" device="C0805" value="10uF"/>
+<part name="C1" library="rcl" deviceset="C-US" device="C0805" value="1uF"/>
 <part name="C2" library="rcl" deviceset="C-US" device="C0805" value="0.1uF"/>
 <part name="R3" library="rcl" deviceset="R-US_" device="R0805" value="68"/>
@@
 <part name="GND4" library="supply1" deviceset="GND" device=""/>
 <part name="P+5" library="supply1" deviceset="VCC" device=""/>
-<part name="R4" library="rcl" deviceset="R-US_" device="R0805" value="4.7K"/>
+<part name="R4" library="rcl" deviceset="R-US_" device="R0805" value="10K"/>
 <part name="ICSP1" library="SparkFun-Connectors" deviceset="AVR_SPI_PRG_6" device="2X3_LOCK"/>
 <part name="LED1" library="weblight" deviceset="APA102" device=""/>
