File: hardware/weblight.brd (EAGLE design)
At the start: 43.2 x 12.7 mm, 16 parts, among them U1 ATtiny85-20SU

Commit message: Checkpoint. Not all routed yet
Parts:
- moved ISP 0.76 mm to (1.14, 6.35)
Routing:
- net N_RESET: track 6.85 -> 32.2 mm, vias 0 -> 1
- net MISO: track 0.00 -> 14.9 mm, vias 0 -> 2
- net CLK_1/SCK: track 6.64 -> 19.9 mm, vias 0 -> 2
- net GND: track 0.00 -> 6.23 mm, vias 0 -> 3
- net VCC: track 47.3 -> 52.3 mm
- net 5V: track 0.00 -> 2.54 mm
- net DIN_1/MOSI: track 18.5 -> 16.5 mm
Changed lines of the file:
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@@
 <attribute name="VALUE" x="8.35" y="6.2336" size="0.8128" layer="27" font="vector" rot="R180" align="top-left"/>
 </element>
-<element name="ISP" library="weblight" package="POGOPROG-CONN-OH-SMALLERVIAS" value="POGOPIN-CONNWITHVIAS-SMV" x="1.905" y="6.35" smashed="yes">
-<attribute name="NAME" x="1.905" y="10.795" size="0.8128" layer="25" font="vector" rot="R270" align="center"/>
-<attribute name="VALUE" x="0.635" y="0" size="1.27" layer="27"/>
+<element name="ISP" library="weblight" package="POGOPROG-CONN-OH-SMALLERVIAS" value="POGOPIN-CONNWITHVIAS-SMV" x="1.143" y="6.35" smashed="yes">
+<attribute name="NAME" x="1.143" y="10.795" size="0.8128" layer="25" font="vector" rot="R270" align="center"/>
+<attribute name="VALUE" x="-0.127" y="0" size="1.27" layer="27"/>
 </element>
 <element name="J-TOP" library="SparkFun-Connectors" package="USB-A-PCB-NOPASTE" value="USBPCB_NOPASTE" x="38.1" y="6.35" smashed="yes" rot="R180">
@@
 <wire x1="13.02" y1="2.54" x2="12.954" y2="2.54" width="0.381" layer="1"/>
 <wire x1="12.954" y1="2.54" x2="12.954" y2="0.762" width="0.6096" layer="1"/>
-<wire x1="12.954" y1="0.762" x2="25.715" y2="0.762" width="0.6096" layer="1"/>
 <wire x1="25.715" y1="0.762" x2="25.715" y2="2.54" width="0.6096" layer="1"/>
 <wire x1="13.02" y1="5.08" x2="11.684" y2="5.08" width="0.6096" layer="1"/>
@@
 <wire x1="8.35" y1="2.032" x2="7.112" y2="2.032" width="0.254" layer="1"/>
 <wire x1="7.112" y1="2.032" x2="7.112" y2="2.54" width="0.254" layer="1"/>
-<wire x1="7.112" y1="2.54" x2="1.905" y2="2.54" width="0.254" layer="1"/>
+<wire x1="7.112" y1="2.54" x2="1.143" y2="2.54" width="0.254" layer="1"/>
+<wire x1="13.02" y1="5.08" x2="12.954" y2="0.762" width="0.4064" layer="1"/>
+<wire x1="12.954" y1="0.762" x2="25.715" y2="0.762" width="0.6096" layer="1"/>
 </signal>
 <signal name="GND">
@@
 <polygon width="0.4064" layer="1" rank="6">
 <vertex x="-0.635" y="13.335"/>
-<vertex x="43.815" y="13.335"/>
-<vertex x="43.815" y="-0.635"/>
+<vertex x="34.036" y="13.335"/>
+<vertex x="34.036" y="-0.635"/>
 <vertex x="-0.635" y="-0.635"/>
 </polygon>
 <polygon width="0.4064" layer="16" rank="6">
 <vertex x="-1.27" y="13.97"/>
-<vertex x="44.45" y="13.97"/>
-<vertex x="44.45" y="-1.27"/>
+<vertex x="34.036" y="13.97"/>
+<vertex x="34.036" y="-1.27"/>
 <vertex x="-1.27" y="-1.27"/>
 </polygon>
 <contactref element="J-BOT" pad="GND"/>
+<via x="19.304" y="3.81" extent="1-16" drill="0.381"/>
+<via x="2.54" y="1.778" extent="1-16" drill="0.381"/>
+<wire x1="2.54" y1="1.778" x2="4.35" y2="1.778" width="0.4064" layer="1"/>
+<wire x1="4.35" y1="1.778" x2="4.35" y2="1.7036" width="0.4064" layer="1"/>
+<wire x1="6.35" y1="1.7036" x2="6.35" y2="1.778" width="0.4064" layer="1"/>
+<wire x1="14.224" y1="1.778" x2="14.986" y2="1.016" width="0.4064" layer="16"/>
+<wire x1="1.143" y1="3.81" x2="2.286" y2="3.81" width="0.4064" layer="1"/>
+<via x="2.286" y="3.81" extent="1-16" drill="0.381"/>
+<wire x1="2.286" y1="3.81" x2="2.54" y2="1.778" width="0.4064" layer="16"/>
 <wire x1="38.3" y1="2.85" x2="38.3" y2="9.85" width="0" layer="19" extent="1-16"/>
-<wire x1="4.35" y1="1.7036" x2="14.92" y2="2.54" width="0" layer="19" extent="1-1"/>
-<wire x1="4.35" y1="7.571" x2="1.905" y2="3.81" width="0" layer="19" extent="1-1"/>
+<wire x1="31.115" y1="10.16" x2="38.3" y2="9.85" width="0" layer="19" extent="1-16"/>
 </signal>
 <signal name="USB_D_MINUS">
@@
 <wire x1="21.336" y1="6.604" x2="21.336" y2="7.366" width="0.381" layer="1"/>
 <wire x1="21.336" y1="7.366" x2="19.2532" y2="7.366" width="0.381" layer="1"/>
-<wire x1="1.905" y1="8.89" x2="19.2532" y2="7.366" width="0" layer="19" extent="1-1"/>
+<wire x1="19.2532" y1="7.366" x2="16.002" y2="7.366" width="0.4064" layer="1"/>
+<via x="16.002" y="7.366" extent="1-16" drill="0.381"/>
+<wire x1="16.002" y1="7.366" x2="15.748" y2="7.366" width="0.4064" layer="16"/>
+<wire x1="15.748" y1="7.366" x2="15.748" y2="11.938" width="0.4064" layer="16"/>
+<wire x1="15.748" y1="11.938" x2="1.778" y2="11.938" width="0.4064" layer="16"/>
+<wire x1="1.778" y1="11.938" x2="1.778" y2="11.684" width="0.4064" layer="16"/>
+<wire x1="1.778" y1="11.684" x2="1.905" y2="11.684" width="0.4064" layer="16"/>
+<wire x1="1.905" y1="11.684" x2="1.143" y2="8.89" width="0.4064" layer="16"/>
 </signal>
 <signal name="CLK_1/SCK">
@@
 <contactref element="LED1" pad="CI"/>
 <contactref element="ISP" pad="4"/>
-<wire x1="4.35" y1="9.271" x2="2.794" y2="9.271" width="0.3048" layer="1"/>
-<wire x1="2.794" y1="9.271" x2="2.794" y2="5.08" width="0.3048" layer="1"/>
-<wire x1="2.794" y1="5.08" x2="1.905" y2="5.08" width="0.3048" layer="1"/>
-<wire x1="4.35" y1="9.271" x2="12.5222" y2="8.636" width="0" layer="19" extent="1-1"/>
+<wire x1="4.35" y1="9.271" x2="2.48285" y2="9.271" width="0.3048" layer="1"/>
+<wire x1="2.48285" y1="9.271" x2="2.48285" y2="5.08" width="0.3048" layer="1"/>
+<wire x1="2.48285" y1="5.08" x2="1.143" y2="5.08" width="0.3048" layer="1"/>
+<wire x1="12.5222" y1="8.636" x2="9.906" y2="8.636" width="0.4064" layer="1"/>
+<via x="9.906" y="8.636" extent="1-16" drill="0.381"/>
+<wire x1="9.906" y1="8.636" x2="4.318" y2="8.636" width="0.4064" layer="16"/>
+<wire x1="4.318" y1="8.636" x2="4.318" y2="10.16" width="0.4064" layer="16"/>
+<wire x1="4.318" y1="10.16" x2="2.48285" y2="10.16" width="0.4064" layer="16"/>
+<via x="2.48285" y="10.16" extent="1-16" drill="0.381"/>
+<wire x1="2.48285" y1="10.16" x2="2.48285" y2="9.271" width="0.254" layer="1"/>
 </signal>
 <signal name="DIN_2">
@@
 <contactref element="ISP" pad="3"/>
 <contactref element="U1" pad="6"/>
-<wire x1="1.905" y1="6.35" x2="12.5222" y2="9.906" width="0" layer="19" extent="1-1"/>
+<wire x1="12.5222" y1="9.906" x2="10.668" y2="9.906" width="0.4064" layer="1"/>
+<via x="10.668" y="9.906" extent="1-16" drill="0.381"/>
+<wire x1="10.668" y1="9.906" x2="10.668" y2="6.35" width="0.4064" layer="16"/>
+<wire x1="10.668" y1="6.35" x2="1.143" y2="6.35" width="0.4064" layer="16"/>
+<via x="1.143" y="6.35" extent="1-16" drill="0.381"/>
 </signal>
 <signal name="DIN_1/MOSI">
@@
 <contactref element="U1" pad="5"/>
 <wire x1="12.5222" y1="11.176" x2="12.446" y2="11.176" width="0.3048" layer="1"/>
-<wire x1="12.446" y1="11.176" x2="12.446" y2="12.192" width="0.3048" layer="1"/>
-<wire x1="12.446" y1="12.192" x2="4.35" y2="12.192" width="0.3048" layer="1"/>
-<wire x1="4.35" y1="12.192" x2="4.35" y2="10.971" width="0.3048" layer="1"/>
-<wire x1="4.35" y1="10.971" x2="0.762" y2="10.971" width="0.3048" layer="1"/>
-<wire x1="0.762" y1="10.971" x2="0.762" y2="7.62" width="0.3048" layer="1"/>
-<wire x1="0.762" y1="7.62" x2="1.905" y2="7.62" width="0.3048" layer="1"/>
+<wire x1="12.446" y1="11.176" x2="12.446" y2="11.938" width="0.3048" layer="1"/>
+<wire x1="12.446" y1="11.938" x2="4.35" y2="11.938" width="0.3048" layer="1"/>
+<wire x1="4.35" y1="11.938" x2="4.35" y2="10.971" width="0.3048" layer="1"/>
+<wire x1="4.35" y1="10.971" x2="1.8288" y2="10.971" width="0.3048" layer="1"/>
+<wire x1="1.8288" y1="10.971" x2="1.8288" y2="7.62" width="0.254" layer="1"/>
+<wire x1="1.8288" y1="7.62" x2="1.143" y2="7.62" width="0.3048" layer="1"/>
 </signal>
 <signal name="5V">
@@
 <contactref element="J-BOT" pad="5V"/>
 <contactref element="D4" pad="A"/>
+<wire x1="31.115" y1="7.62" x2="31.115" y2="5.08" width="0.4064" layer="1"/>
 <wire x1="38.3" y1="2.85" x2="38.3" y2="9.85" width="0" layer="19" extent="1-16"/>
 <wire x1="31.115" y1="7.62" x2="38.3" y2="9.85" width="0" layer="19" extent="1-1"/>
-<wire x1="31.115" y1="5.08" x2="31.115" y2="7.62" width="0" layer="19" extent="1-1"/>
 </signal>
 </signals>

Commit message: Checkpoint #2, all but connectors
Routing:
- net USB_D_MINUS_RAW: track 1.14 -> 14.2 mm, vias 0 -> 3
Changed lines of the file:
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@@
 <contactref element="J-TOP" pad="USB_M"/>
 <contactref element="J-BOT" pad="USB_M"/>
-<wire x1="28.575" y1="2.54" x2="27.432" y2="2.54" width="0.381" layer="1"/>
+<wire x1="28.575" y1="2.54" x2="27.178" y2="2.54" width="0.4064" layer="1"/>
+<via x="27.178" y="2.54" extent="1-16" drill="0.381"/>
+<wire x1="27.178" y1="2.54" x2="22.352" y2="2.54" width="0.4064" layer="16"/>
+<via x="22.352" y="2.54" extent="1-16" drill="0.381"/>
+<wire x1="22.352" y1="2.54" x2="23.815" y2="2.54" width="0.4064" layer="1"/>
+<wire x1="25.715" y1="7.62" x2="27.178" y2="7.62" width="0.4064" layer="1"/>
+<via x="27.178" y="7.62" extent="1-16" drill="0.381"/>
+<wire x1="27.178" y1="7.62" x2="27.178" y2="2.54" width="0.4064" layer="16"/>
 <wire x1="37.8" y1="5.35" x2="37.8" y2="7.35" width="0" layer="19" extent="1-16"/>
 <wire x1="28.575" y1="2.54" x2="37.8" y2="5.35" width="0" layer="19" extent="1-16"/>
-<wire x1="23.815" y1="2.54" x2="27.432" y2="2.54" width="0" layer="19" extent="1-1"/>
-<wire x1="25.715" y1="7.62" x2="27.432" y2="2.54" width="0" layer="19" extent="1-1"/>
 </signal>
 <signal name="USB_D_PLUS_RAW">
